Commit message: Added models and files

File: models/rotors_description/urdf/component_snippets.xacro (robot description, xacro)
@@ -50,5 +50,4 @@
             <xacro:insert_block name="cylinder" />
           </geometry>
-          <material name="red" />
         </visual>
       </xacro:if>
@@ -65,4 +64,5 @@
     </joint>
     <gazebo reference="${namespace}/camera_${camera_suffix}_link">
+      <material>Gazebo/Yellow</material>
       <sensor type="camera" name="${namespace}_camera_${camera_suffix}">
         <update_rate>${frame_rate}</update_rate>
@@ -486,5 +486,5 @@
       noise_mean="0.0"
       noise_stddev="0.007"
-      enable_visual="false">
+      enable_visual="true">
       <cylinder length="0.01" radius="0.007" />
       <xacro:insert_block name="origin" />
@@ -498,7 +498,13 @@
         <origin xyz="0 0 0" rpy="0 0 0" />
         <geometry>
-          <cylinder length="0.01" radius="0.007" />
+          <cylinder length="0.02" radius="0.005" />
         </geometry>
       </collision>
+      <visual>
+        <origin xyz="0 0 0" rpy="0 0 0" />
+        <geometry>
+          <cylinder length="0.02" radius="0.005" />
+        </geometry>
+      </visual>
       <inertial>
         <mass value="1e-5" />
@@ -516,5 +522,5 @@
     <link name="${namespace}/camera_${camera_suffix}_optical_center_link" />
     <joint name="${namespace}/camera_${camera_suffix}_optical_center_joint" type="fixed">
-      <origin xyz="0 0 0" rpy="${-PI/2} 0 ${-PI/2}" />
+      <origin xyz="0 0 0" rpy="${-3.14159265359/2} 0 ${-3.14159265359/2}" />
       <parent link="${namespace}/camera_${camera_suffix}_link" />
       <child link="${namespace}/camera_${camera_suffix}_optical_center_link" />
@@ -522,9 +528,14 @@
     </joint>
     <gazebo reference="${namespace}/camera_${camera_suffix}_link">
-      <sensor type="depth" name="${namespace}_camera_{camera_suffix}">
+      <material>Gazebo/Green</material>
+<!--      <sensor type="depth" name="${namespace}_camera_{camera_suffix}">
         <always_on>true</always_on>
         <update_rate>${frame_rate}</update_rate>
         <camera>
           <horizontal_fov>2</horizontal_fov>
+          <ray>
+            <horizontal samples="100" resolution="1" min_angle="-1.5708" max_angle="1.5708"/>
+            <vertical samples="1" resolution="1" min_angle="0" max_angle="0"/>
+          </ray>
           <image>
             <format>L8</format>
@@ -555,4 +566,38 @@
           <distortionT1>0.0</distortionT1>
           <distortionT2>0.0</distortionT2>
+        </plugin>
+      </sensor> -->
+<!-- newly added -->
+      <sensor type="ray" name="${namespace}_camera_{camera_suffix}">
+        <always_on>1</always_on>
+        <update_rate>40</update_rate>
+        <visualize>true</visualize>
+        <ray>
+          <scan>
+            <horizontal>
+              <samples>720</samples>
+              <resolution>1</resolution>
+              <min_angle>-1.26889</min_angle>
+              <max_angle>1.268899</max_angle>
+            </horizontal>
+          </scan>
+          <range>
+            <min>0.08</min>
+            <max>30</max>
+            <resolution>0.01</resolution>
+          </range>
+          <noise>
+            <type>gaussian</type>
+      <!-- Noise parameters based on published spec for Hokuyo laser
+           achieving "+-30mm" accuracy at range < 10m.  A mean of 0.0m and
+           stddev of 0.01m will put 99.7% of samples within 0.03m of the true
+           reading. -->
+            <mean>0.0</mean>
+            <stddev>0.01</stddev>
+          </noise>
+        </ray>
+        <plugin name="${namespace}_camera_{camera_suffix}" filename="libgazebo_ros_laser.so">
+          <robotNamespace>${namespace}</robotNamespace>
+          <topicName>${camera_suffix}</topicName>
         </plugin>
       </sensor>

File: models/rotors_description/urdf/iris_base.xacro (robot description, xacro)
@@ -29,4 +29,5 @@
   <xacro:arg name='enable_logging' default='false' />
   <xacro:arg name='log_file' default='iris' />
+  <xacro:arg name='enable_depth' default='true' />
   <!-- macros for gazebo plugins, sensors -->
   <xacro:include filename="$(arg rotors_description_dir)/urdf/component_snippets.xacro" />
@@ -96,4 +97,38 @@
   </xacro:mavlink_interface_macro>
   </xacro:if>
+  <!-- Mount a camera -->
+  <!--<xacro:vi_sensor_camera_macro
+  namespace="${namespace}"
+  parent_link="base_link"
+  camera_suffix="red_iris"
+  frame_rate="60.0"
+  >
+  <box size="0.05 0.05 0.05" />
+  <origin xyz="0 0 0.05" rpy="0 0 0"/>
+  </xacro:vi_sensor_camera_macro>-->
+  <xacro:vi_sensor_depth_macro
+  namespace="${namespace}" parent_link="base_link"
+  camera_suffix="hokuyo_scan" frame_rate="40.0">
+  <origin xyz="0 0 -0.05" rpy="0 1.57079 0"/>
+  </xacro:vi_sensor_depth_macro>
+   <!-- Mount a camera -->
+  <xacro:camera_macro
+  namespace="${namespace}"
+  parent_link="base_link"
+  camera_suffix="red_iris"
+  frame_rate="30.0"
+  horizontal_fov="1.3962634"
+  image_width="800"
+  image_height="800"
+  image_format="R8G8B8"
+  min_distance="0.02"
+  max_distance="10"
+  noise_mean="0.0"
+  noise_stddev="0.007"
+  enable_visual="1"
+  >
+  <box size="0.05 0.05 0.05" />
+  <origin xyz="0 0 0.05" rpy="0 0 0"/>
+  </xacro:camera_macro>-->
   <!-- Mount an ADIS16448 IMU. -->
   <xacro:imu_plugin_macro

Commit message: Latest Commit from Melodic

File: models/rotors_description/urdf/component_snippets.xacro (robot description, xacro)
@@ -529,5 +529,5 @@
     <gazebo reference="${namespace}/camera_${camera_suffix}_link">
       <material>Gazebo/Green</material>
-<!--      <sensor type="depth" name="${namespace}_camera_{camera_suffix}">
+      <sensor type="depth" name="${namespace}_camera_{camera_suffix}">
         <always_on>true</always_on>
         <update_rate>${frame_rate}</update_rate>
@@ -572,5 +572,5 @@
         <always_on>1</always_on>
         <update_rate>40</update_rate>
-        <visualize>true</visualize>
+        <visualize>false</visualize>
         <ray>
           <scan>

File: models/rotors_description/urdf/iris_base.xacro (robot description, xacro)
@@ -110,5 +110,6 @@
   namespace="${namespace}" parent_link="base_link"
   camera_suffix="hokuyo_scan" frame_rate="40.0">
-  <origin xyz="0 0 -0.05" rpy="0 1.57079 0"/>
+  <!--<origin xyz="0 0 -0.05" rpy="0 1.57079 0"/> UPSIDE DOWN -->
+  <origin xyz="0 0 0.09" rpy="0 0 0"/>
   </xacro:vi_sensor_depth_macro>
    <!-- Mount a camera -->
@@ -129,5 +130,5 @@
   >
   <box size="0.05 0.05 0.05" />
-  <origin xyz="0 0 0.05" rpy="0 0 0"/>
+  <origin xyz="0 0 0.05" rpy="0 0 3.1416"/>
   </xacro:camera_macro>-->
   <!-- Mount an ADIS16448 IMU. -->

File: models/rotors_description/urdf/iris_base_head.xacro (robot description, xacro)
@@ -31,7 +31,7 @@
   <xacro:arg name='enable_depth' default='true' />
   <!-- macros for gazebo plugins, sensors -->
-  <xacro:include filename="$(arg rotors_description_dir)/urdf/component_snippets.xacro" />
+  <xacro:include filename="$(arg rotors_description_dir)/urdf/component_snippets_head.xacro" />
   <!-- Instantiate iris "mechanics" -->
-  <xacro:include filename="$(arg rotors_description_dir)/urdf/iris.xacro" />
+  <xacro:include filename="$(arg rotors_description_dir)/urdf/iris_head.xacro" />
   <xacro:if value="$(arg enable_wind)">
     <xacro:wind_plugin_macro
@@ -97,9 +97,34 @@
   </xacro:mavlink_interface_macro>
   </xacro:if>
+  <xacro:vi_sensor_depth_macro
+  namespace="${namespace}" parent_link="fcu"
+  camera_suffix="structure_core" frame_rate="40.0">
+  <!--<origin xyz="0 0 -0.05" rpy="0 1.57079 0"/> UPSIDE DOWN -->
+  <origin xyz="0 0 0.09" rpy="0 0 0"/>
+  </xacro:vi_sensor_depth_macro>
+   <!-- Mount a camera -->
+  <xacro:camera_macro
+  namespace="${namespace}"
+  parent_link="fcu"
+  camera_suffix="non_red_iris"
+  frame_rate="30.0"
+  horizontal_fov="1.3962634"
+  image_width="800"
+  image_height="800"
+  image_format="R8G8B8"
+  min_distance="0.02"
+  max_distance="10"
+  noise_mean="0.0"
+  noise_stddev="0.007"
+  enable_visual="1"
+  >
+  <box size="0.05 0.05 0.05" />
+  <origin xyz="0 0 0.05" rpy="0 0 3.1416"/>
+  </xacro:camera_macro>-->
   <!-- Mount an ADIS16448 IMU. -->
   <xacro:imu_plugin_macro
     namespace="${namespace}"
     imu_suffix=""
-    parent_link="base_link"
+    parent_link="fcu"
     imu_topic="/imu"
     mass_imu_sensor="0.015"
@@ -121,5 +146,5 @@
       namespace="${namespace}"
       imu_suffix="gt"
-      parent_link="base_link"
+      parent_link="fcu"
       imu_topic="ground_truth/imu"
       mass_imu_sensor="0.00001"
@@ -140,5 +165,5 @@
       namespace="${namespace}/ground_truth"
       odometry_sensor_suffix="gt"
-      parent_link="base_link"
+      parent_link="fcu"
       pose_topic="pose"
       pose_with_covariance_topic="pose_with_covariance"
